File: cnc-grbl.sch (KiCad schematic (older format))
At the start: 61 parts, among them IC1 ATMEGA328P-A, P1 ICSP, P10 Z MOT, P11 CTR, P12 CON, P13 CONN_02X03, P2 USB_B, P3 CONN_02X03, P4 CONN_02X03, P5 CONN_02X03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

Commit message: pcb tested and working
Parts:
- P2: symbol USB_B -> USB_B-RESCUE-cnc-grbl
Changed lines of the file:
@@
 EESchema Schematic File Version 2
+LIBS:cnc-grbl-rescue
 LIBS:valves
 LIBS:power
@@
 $EndComp
 $Comp
-L USB_B P2
+L USB_B-RESCUE-cnc-grbl P2
 U 1 1 57B3BD66
 P 6575 6950
